File: DIY_Keyboard/DIY_Keyboard_V1.brd (EAGLE design)
At the start: 322 x 94 mm, 171 parts, among them Y1 16MHz

Commit message: Updated Files
Routing:
- net GND: track 465.1 -> 468.7 mm
- net R4: track 358.4 -> 360.7 mm
- net C12: track 167.2 -> 169.3 mm
- net N$88: track 274.5 -> 272.8 mm
- net C7: track 252.2 -> 253.7 mm
- net C14: track 145.1 -> 146.2 mm
- net R5: track 373.3 -> 374.3 mm
- net R1: track 336.1 -> 337.0 mm
- net N$90: track 112.0 -> 112.9 mm
- net R2: track 315.0 -> 315.7 mm
- net N$83: track 271.3 -> 272.0 mm
- net N$89: track 107.6 -> 108.3 mm
Other:
- board text added: "AForland"
- board text added: "C:/Users/tankh/Pictures/ShelbyTech.bmp"
- board text added: "Thanks for the help!!"
- board text removed: "Mech-E_V1.0"
- board text removed: "Shelby_Tech\"
