File: DIY_Keyboard_V1.1/DIY_Keyboard_V1.1.brd (EAGLE design)
At the start: 322 x 94 mm, 176 parts, among them Y1 16MHz

Commit message: Updated connections
Cleared all airwire and clearance errors
Routing:
- net N$90: track 0.00 -> 209.1 mm, vias 0 -> 8
- net N$93: track 0.00 -> 180.0 mm, vias 0 -> 6
- net N$92: track 0.00 -> 86.9 mm, vias 0 -> 4
- net VCC: track 272.0 -> 337.4 mm, vias 7 -> 8
- net N$88: track 272.8 -> 336.5 mm, vias 4 -> 7
- net N$85: track 33.5 -> 87.8 mm, vias 1 -> 4
- net GND: track 468.7 -> 508.6 mm, vias 9 -> 13
- net N$89: track 108.3 -> 131.3 mm, vias 2 -> 5
- net C12: track 172.4 -> 190.8 mm
- net C17: track 165.7 -> 178.8 mm
- net N$87: track 77.1 -> 80.8 mm
- net N$82: track 125.8 -> 128.1 mm
- net N$84: track 155.3 -> 153.8 mm
- net C1: track 312.8 -> 313.9 mm
- net N$86: track 57.6 -> 58.7 mm
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Other:
- board text added: "RST"

Commit message: Version 1.1 done!!
Parts:
- R3, R4: value 56k -> 5.1k
Changed lines of the file:
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@@
 </element>
 <element name="U$1" library="USB-TYPE-C-V2" package="USB_TYPE_C" value="USB_TYPE_C" x="-303.5" y="17" smashed="yes" rot="R180"/>
-<element name="R3" library="SparkFun-Resistors" package="0603" value="56k" x="-226" y="-46.5" smashed="yes">
+<element name="R3" library="SparkFun-Resistors" package="0603" value="5.1k" x="-226" y="-46.5" smashed="yes">
 <attribute name="NAME" x="-226" y="-45.738" size="0.6096" layer="25" font="vector" ratio="20" align="bottom-center"/>
 <attribute name="VALUE" x="-226" y="-47.262" size="0.6096" layer="27" font="vector" ratio="20" align="top-center"/>
 </element>
-<element name="R4" library="SparkFun-Resistors" package="0603" value="56k" x="-226" y="-49" smashed="yes">
+<element name="R4" library="SparkFun-Resistors" package="0603" value="5.1k" x="-226" y="-49" smashed="yes">
 <attribute name="NAME" x="-226" y="-48.238" size="0.6096" layer="25" font="vector" ratio="20" align="bottom-center"/>
 <attribute name="VALUE" x="-226" y="-49.762" size="0.6096" layer="27" font="vector" ratio="20" align="top-center"/>
