File: DIY_Keyboard_V1.4/DIY_Keyboard_V1.4.brd (EAGLE design)
At the start: 322 x 94 mm, 171 parts, among them Y1 16MHz

Commit message: Update board files
Parts:
- moved U$1 14.7 mm to (-302.7, 31.7)
Routing:
- net R1: track 337.0 -> 40.3 mm, vias 1 -> 0
- net C16: track 282.7 -> 14.4 mm, vias 2 -> 0
- net VCC: track 294.3 -> 43.4 mm, vias 7 -> 0
- net GND: track 289.8 -> 86.9 mm, vias 11 -> 0
- net C10: track 221.3 -> 32.2 mm, vias 2 -> 0
- net C7: track 253.7 -> 80.2 mm, vias 2 -> 0
- net C12: track 190.8 -> 26.9 mm, vias 5 -> 0
- net R2: track 315.7 -> 160.8 mm, vias 1 -> 0
- net C9: track 192.8 -> 52.4 mm, vias 4 -> 0
- net C11: track 144.5 -> 8.28 mm, vias 3 -> 0
- net C6: track 223.9 -> 95.0 mm, vias 4 -> 0
- net N$82: track 128.1 -> 0.00 mm
- net C17: track 178.8 -> 52.4 mm, vias 4 -> 0
- net C13: track 180.6 -> 65.8 mm, vias 4 -> 0
- net R3: track 364.7 -> 252.1 mm, vias 4 -> 0
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- removed copper zone on layer 1, net GND
Other:
- board size 322 x 94 mm -> 9.3 x 5.7 mm
- board text removed: "AForland"
- board text removed: "C:/Users/tankh/Pictures/ShelbyTech.bmp"
- board text removed: "Capacitor_Land"
- board text removed: "GND"
- board text removed: "MISO"
- board text removed: "MOSI"
- board text removed: "RST"
- board text removed: "Resistor_Land"
- board text removed: "SCK"
- board text removed: "Thanks for the help!!"
- board text removed: "VCC"

Commit message: update board layout
Parts:
- moved S69 523.5 mm to (-435.6, 290.8), turned to 0 degrees
- moved S70 498.1 mm to (-419.1, 290.8), turned to 0 degrees
- moved S51 487.8 mm to (-402.6, 250.2), turned to 0 degrees
- moved S71 469.6 mm to (-402.6, 290.8), turned to 0 degrees
- moved S52 455.0 mm to (-386.1, 250.2), turned to 0 degrees
- moved S67 445.4 mm to (-303.5, 270.5), turned to 0 degrees
- moved D67 443.0 mm to (-232.4, 327.7)
- moved D68 435.6 mm to (-238.8, 327.7)
- moved S79 434.2 mm to (-97.8, 311.1), turned to 0 degrees
- moved S72 433.9 mm to (-386.1, 290.8), turned to 0 degrees
- moved S39 430.8 mm to (-435.6, 229.9), turned to 0 degrees
- moved D69 429.7 mm to (-245.1, 327.7)
- moved S53 428.8 mm to (-369.6, 250.2), turned to 0 degrees
- moved D70 424.2 mm to (-251.5, 327.7)
- moved D79 424.1 mm to (-137.2, 331.5)
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Routing:
- net R5: track 291.0 -> 0.00 mm
- net R4: track 257.1 -> 0.00 mm
- net R3: track 252.1 -> 0.00 mm
- net C1: track 226.2 -> 0.00 mm
- net C2: track 219.5 -> 0.00 mm
- net N$88: track 200.5 -> 0.00 mm
- net C4: track 194.7 -> 0.00 mm
- net C3: track 177.9 -> 0.00 mm
- net R2: track 160.8 -> 0.00 mm
- net N$84: track 131.9 -> 0.00 mm
- net C5: track 129.5 -> 0.00 mm
- net C15: track 98.9 -> 0.00 mm
- net C6: track 95.0 -> 0.00 mm
- net GND: track 86.9 -> 0.00 mm
- net N$89: track 83.6 -> 0.00 mm
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- removed copper zone on layer 16, net GND
Other:
- board size 9.3 x 5.7 mm -> 329.8 x 101.2 mm
- board text removed: "RES"

Commit message: Working on pcb layout
Parts:
- moved S69 755.7 mm to (261.9, 0.00), turned to 180 degrees
- moved S51 737.4 mm to (297.7, 19.1), turned to 180 degrees
- moved S70 723.1 mm to (242.9, 0.00), turned to 180 degrees
- moved S52 697.0 mm to (271.5, 19.1), turned to 180 degrees
- moved S39 686.8 mm to (223.8, 38.1), turned to 180 degrees
- moved S71 684.2 mm to (216.7, 0.00), turned to 180 degrees
- moved S67 663.6 mm to (302.4, 0.00), turned to 180 degrees
- moved S53 663.5 mm to (252.4, 19.1), turned to 180 degrees
- moved S40 652.7 mm to (204.8, 38.1), turned to 180 degrees
- moved S72 630.9 mm to (173.8, 0.00), turned to 180 degrees
- moved S54 630.3 mm to (233.4, 19.1), turned to 180 degrees
- moved S68 629.1 mm to (281.0, 0.00), turned to 180 degrees
- moved S59 626.4 mm to (138.1, 19.1), turned to 180 degrees
- moved S36 625.0 mm to (281.0, 38.1), turned to 180 degrees
- moved S41 618.8 mm to (185.7, 38.1), turned to 180 degrees
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
Commit message: update layout
Parts:
- moved D1 514.9 mm to (304.8, 66.7)
- moved D2 503.7 mm to (285.8, 66.7)
- moved D3 492.5 mm to (266.7, 66.7)
- moved D4 481.4 mm to (247.7, 66.7)
- moved C1 393.8 mm to (191.1, 121.9)
- moved C2 393.8 mm to (187.3, 121.9)
- moved C3 393.8 mm to (183.5, 121.9)
- moved C4 393.8 mm to (179.7, 121.9)
- moved D10 393.8 mm to (123.8, 94.0)
- moved D11 393.8 mm to (117.5, 94.0)
- moved D12 393.8 mm to (111.1, 94.0)
- moved D13 393.8 mm to (104.8, 94.0)
- moved D14 393.8 mm to (98.4, 94.0)
- moved D15 393.8 mm to (92.1, 94.0)
- moved D16 393.8 mm to (85.7, 94.0)
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
Commit message: Update layout
Parts:
- moved D67 229.5 mm to (302.4, 8.10)
- moved D50 227.3 mm to (0.00, 28.6)
- moved D79 226.8 mm to (0.00, 8.10)
- moved D68 216.4 mm to (281.0, 8.10)
- moved D78 215.9 mm to (19.1, 8.10)
- moved D49 215.7 mm to (19.1, 28.6)
- moved D69 205.6 mm to (261.9, 8.10)
- moved D48 204.2 mm to (38.1, 28.6)
- moved D77 197.4 mm to (47.6, 8.10)
- moved D70 195.0 mm to (242.9, 8.10)
- moved D47 192.9 mm to (57.1, 28.6)
- moved D35 190.1 mm to (302.4, 28.6)
- moved D71 178.9 mm to (216.7, 8.10)
- moved D76 177.9 mm to (78.6, 8.10)
- moved D36 176.8 mm to (281.0, 28.6)
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Other:
- board size 329.8 x 101.2 mm -> 323.8 x 95.2 mm

Commit message: Updated PCB Layout
Parts:
- moved U$1 212.3 mm to (9.53, 84.3), turned to 180 degrees
- moved R2 171.9 mm to (7.14, 73.3)
- moved R1 171.5 mm to (11.4, 73.3)
- moved R3 169.9 mm to (6.19, 71.0), turned to 180 degrees
- moved R4 160.4 mm to (12.4, 71.0), turned to 180 degrees
- moved C1 115.7 mm to (205.4, 7.14)
- moved C2 115.7 mm to (201.6, 7.14)
- moved C3 115.7 mm to (197.8, 7.14)
- moved C4 115.7 mm to (194.0, 7.14)
- moved ISP 66.7 mm to (177.0, 29.1), turned to 90 degrees
Routing:
- net GND: track 0.00 -> 439.7 mm, vias 0 -> 10
- net R1: track 0.00 -> 377.7 mm
- net R2: track 0.00 -> 374.3 mm, vias 0 -> 2
- net VCC: track 0.00 -> 354.3 mm, vias 0 -> 7
- net R3: track 0.00 -> 334.4 mm
- net R4: track 0.00 -> 314.9 mm, vias 0 -> 1
- net R5: track 0.00 -> 314.8 mm, vias 0 -> 1
- net C13: track 0.00 -> 308.3 mm, vias 0 -> 6
- net C3: track 0.00 -> 302.7 mm, vias 0 -> 3
- net C16: track 0.00 -> 290.6 mm, vias 0 -> 5
- net C15: track 0.00 -> 268.1 mm, vias 0 -> 4
- net C12: track 0.00 -> 250.5 mm, vias 0 -> 4
- net C17: track 0.00 -> 234.8 mm, vias 0 -> 2
- net C2: track 0.00 -> 234.2 mm, vias 0 -> 3
- net C1: track 0.00 -> 233.2 mm, vias 0 -> 2
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- added copper zone on layer 1, net GND
- added copper zone on layer 16, net GND
