File: DIY_Keyboard_V1.4/DIY_Keyboard_V1.4.brd (EAGLE design)
At the start: 323.8 x 95.2 mm, 171 parts, among them Y1 16MHz

Commit message: Update pcb layout and reexport gerber
Routing:
- net GND: track 439.7 -> 440.6 mm
